Commit message: fix the rviz2 robot model diplay issue

File: igt_ignition/models/igt_one/igt_one.urdf (robot description, URDF)
Before this commit: robot igt_one, 16 links, 15 joints
Links:
- link base_link: geometry collision mesh filename=package://igt_ignition/models/igt_one/meshes/base_link.stl scale=0.001 0.001 0.001; visual mesh filename=package://igt_ignition/models/igt_one/meshes/base_link.stl scale=0.001 0.001 0.001
- link caster_back: geometry collision mesh filename=package://igt_ignition/models/igt_one/meshes/caster_back.stl scale=0.001 0.001 0.001; visual mesh filename=package://igt_ignition/models/igt_one/meshes/caster_back.stl scale=0.001 0.001 0.001
- link caster_front: geometry collision mesh filename=package://igt_ignition/models/igt_one/meshes/caster_front.s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 scale=0.001 0.001 0.001; visual mesh filename=package://igt_ignition/models/igt_one/meshes/caster_front.s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 scale=0.001 0.001 0.001
- link d435_link: geometry collision box size=0.02505 0.09 0.025; visual mesh filename=package://igt_ignition/models/igt_one/meshes/realsense_d435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
- link left_wheel: geometry collision mesh filename=package://igt_ignition/models/igt_one/meshes/left_wheel.stl scale=0.001 0.001 0.001; visual mesh filename=package://igt_ignition/models/igt_one/meshes/left_wheel.stl scale=0.001 0.001 0.001
- link lidar: geometry collision mesh filename=package://igt_ignition/models/igt_one/meshes/lidar.stl scale=0.001 0.001 0.001; visual mesh filename=package://igt_ignition/models/igt_one/meshes/lidar.stl scale=0.001 0.001 0.001
- link right_wheel: geometry collision mesh filename=package://igt_ignition/models/igt_one/meshes/right_wheel.stl scale=0.001 0.001 0.001; visual mesh filename=package://igt_ignition/models/igt_one/meshes/right_wheel.stl scale=0.001 0.001 0.001
